Commit message: update launch and xacro files

File: unitree_go2_description/urdf/unitree_go2_gazebo.xacro (robot description, xacro)
@@ -1,4 +1,5 @@
 <?xml version="1.0"?>
-<robot>
+<robot xmlns:xacro="http://ros.org/wiki/xacro">
+<xacro:macro name="unitree_go2_gazebo" params="robot_controllers">
   <!-- Gazebo Sim plugins -->
   <gazebo>
@@ -25,5 +26,5 @@
   <gazebo>
     <plugin filename="gz_ros2_control-system" name="gz_ros2_control::GazeboSimROS2ControlPlugin">
-      <parameters>$(find unitree_go2_sim)/config/ros_control/ros_control.yaml</parameters>
+      <parameters>${robot_controllers}</parameters>
       <robot_param_node>robot_state_publisher</robot_param_node>
     </plugin>
@@ -218,3 +219,4 @@
     <kd>1.0</kd>
   </gazebo>
+</xacro:macro>
 </robot>

File: unitree_go2_description/urdf/unitree_go2_robot.xacro (robot description, xacro)
@@ -3,4 +3,5 @@
     xmlns:xacro="http://www.ros.org/wiki/xacro">
     <xacro:arg name="DEBUG" default="false"/>
+    <xacro:arg name="robot_controllers" default="$(find unitree_go2_sim)/config/ros_control/ros_control.yaml"/>
     <xacro:include filename="$(find unitree_go2_description)/urdf/const.xacro"/>
     <xacro:include filename="$(find unitree_go2_description)/urdf/materials.xacro"/>
@@ -12,4 +13,5 @@
     <xacro:include filename="$(find unitree_go2_description)/urdf/lidar_4D_lidar.xacro"/>
     <!-- <xacro:stairs stairs="15" xpos="0" ypos="0" zpos="0" /> -->
+    <xacro:unitree_go2_gazebo robot_controllers="$(arg robot_controllers)"/>
     <!-- Rotor related joint and link is only for demonstrate location. -->
     <!-- Actually, the rotor will rotate and the joint is not fixed. Reduction ratio should be considered. -->
