Commit message: Disable gz_ros2_control, fix launch headless flags, update LiDAR specs, add disaster world

File: unitree_go2_description/urdf/lidar_4D_lidar.xacro (robot description, xacro)
@@ -1,10 +1,15 @@
 <?xml version="1.0"?>
 <robot xmlns:xacro="http://www.ros.org/wiki/xacro">
-    <!-- Lidar L1-->
+    <!-- Unitree 4D LiDAR L1 — matched to real specs:
+         FOV: 360° horizontal x 90° vertical
+         Range: 0.05m - 30m
+         Samples: 600 horizontal x 90 vertical (~real density)
+         Rate: 11Hz (real circumferential scan frequency)
+         Noise: gaussian stddev 0.02m (matches ±2cm accuracy spec) -->
     <link name="lidar_l1_link">
         <inertial>
-            <mass value="0.5"/>
+            <mass value="0.27"/>
             <origin rpy="0 0 0" xyz="0 0 0"/>
-            <inertia ixx="0.01" ixy="0" ixz="0" iyy="0.01" iyz="0" izz="0.01"/>
+            <inertia ixx="0.001" ixy="0" ixz="0" iyy="0.001" iyz="0" izz="0.001"/>
         </inertial>
         <visual>
@@ -20,21 +25,18 @@
             <origin rpy="0 0 0" xyz="0 0 0"/>
             <geometry>
-                <mesh filename="file://$(find unitree_go2_description)/meshes/L1_4D_Lidar.dae" scale="1 1 1"/>
+                <cylinder radius="0.05" length="0.07"/>
             </geometry>
-            <material name="black">
-                <color rgba="0.0 0.0 0.0 1.0"/>
-            </material>
         </collision>
     </link>
     <joint name="lidar_l1_joint" type="fixed">
-        <parent link="base_link"/>
+        <parent link="trunk"/>
         <child link="lidar_l1_link"/>
-        <!-- <origin rpy="2.94 0 1.5705" xyz="0.25 -0.038 -0.03"/> -->
-        <origin rpy="2.879 0.0 1.5705" xyz="0.25 -0.038 -0.03"/>
+        <!-- Mounted on top-centre of trunk, slightly forward -->
+        <origin rpy="0 0 0" xyz="0.05 0.0 0.12"/>
     </joint>
     <gazebo reference="lidar_l1_link">
         <sensor name="lidar_l1" type="gpu_lidar">
             <topic>unitree_lidar</topic>
-            <update_rate>10</update_rate>
+            <update_rate>11</update_rate>
             <lidar>
                 <scan>
@@ -46,5 +48,5 @@
                     </horizontal>
                     <vertical>
-                        <samples>30</samples>
+                        <samples>90</samples>
                         <resolution>1</resolution>
                         <min_angle>-0.785398</min_angle>
@@ -53,12 +55,12 @@
                 </scan>
                 <range>
-                    <min>0.8</min>
+                    <min>0.05</min>
                     <max>30.0</max>
-                    <resolution>0.001</resolution>
+                    <resolution>0.02</resolution>
                 </range>
                 <noise>
                     <type>gaussian</type>
                     <mean>0.0</mean>
-                    <stddev>0.008</stddev>
+                    <stddev>0.02</stddev>
                 </noise>
             </lidar>

File: unitree_go2_description/urdf/unitree_go2_gazebo.xacro (robot description, xacro)
@@ -24,5 +24,5 @@
         </gazebo> -->
   <!-- ROS2 Control plugin -->
-  <gazebo>
+ <!-- <gazebo>
     <plugin filename="gz_ros2_control-system" name="gz_ros2_control::GazeboSimROS2ControlPlugin">
       <parameters>${robot_controllers}</parameters>
@@ -30,4 +30,5 @@
     </plugin>
   </gazebo>
+-->
         <!-- Odometry plugin -->
         <gazebo>
@@ -220,4 +221,138 @@
     <kd>1.0</kd>
   </gazebo>
+  <!-- Native joint position controllers for direct Gazebo control -->
+  <gazebo>
+    <plugin filename="gz-sim-joint-position-controller-system"
+            name="gz::sim::systems::JointPositionController">
+      <joint_name>lf_hip_joint</joint_name>
+      <p_gain>200</p_gain>
+      <i_gain>0.01</i_gain>
+      <d_gain>10</d_gain>
+      <cmd_max>33.5</cmd_max>
+      <cmd_min>-33.5</cmd_min>
+    </plugin>
+  </gazebo>
+  <gazebo>
+    <plugin filename="gz-sim-joint-position-controller-system"
+            name="gz::sim::systems::JointPositionController">
+      <joint_name>lf_upper_leg_joint</joint_name>
+      <p_gain>200</p_gain>
+      <i_gain>0.01</i_gain>
+      <d_gain>10</d_gain>
+      <cmd_max>33.5</cmd_max>
+      <cmd_min>-33.5</cmd_min>
+    </plugin>
+  </gazebo>
+  <gazebo>
+    <plugin filename="gz-sim-joint-position-controller-system"
+            name="gz::sim::systems::JointPositionController">
+      <joint_name>lf_lower_leg_joint</joint_name>
+      <p_gain>200</p_gain>
+      <i_gain>0.01</i_gain>
+      <d_gain>10</d_gain>
+      <cmd_max>33.5</cmd_max>
+      <cmd_min>-33.5</cmd_min>
+    </plugin>
+  </gazebo>
+  <gazebo>
+    <plugin filename="gz-sim-joint-position-controller-system"
+            name="gz::sim::systems::JointPositionController">
+      <joint_name>rf_hip_joint</joint_name>
+      <p_gain>200</p_gain>
+      <i_gain>0.01</i_gain>
+      <d_gain>10</d_gain>
+      <cmd_max>33.5</cmd_max>
+      <cmd_min>-33.5</cmd_min>
+    </plugin>
+  </gazebo>
+  <gazebo>
+    <plugin filename="gz-sim-joint-position-controller-system"
+            name="gz::sim::systems::JointPositionController">
+      <joint_name>rf_upper_leg_joint</joint_name>
+      <p_gain>200</p_gain>
+      <i_gain>0.01</i_gain>
+      <d_gain>10</d_gain>
+      <cmd_max>33.5</cmd_max>
+      <cmd_min>-33.5</cmd_min>
+    </plugin>
+  </gazebo>
+  <gazebo>
+    <plugin filename="gz-sim-joint-position-controller-system"
+            name="gz::sim::systems::JointPositionController">
+      <joint_name>rf_lower_leg_joint</joint_name>
+      <p_gain>200</p_gain>
+      <i_gain>0.01</i_gain>
+      <d_gain>10</d_gain>
+      <cmd_max>33.5</cmd_max>
+      <cmd_min>-33.5</cmd_min>
+    </plugin>
+  </gazebo>
+  <gazebo>
+    <plugin filename="gz-sim-joint-position-controller-system"
+            name="gz::sim::systems::JointPositionController">
+      <joint_name>lh_hip_joint</joint_name>
+      <p_gain>200</p_gain>
+      <i_gain>0.01</i_gain>
+      <d_gain>10</d_gain>
+      <cmd_max>33.5</cmd_max>
+      <cmd_min>-33.5</cmd_min>
+    </plugin>
+  </gazebo>
+  <gazebo>
+    <plugin filename="gz-sim-joint-position-controller-system"
+            name="gz::sim::systems::JointPositionController">
+      <joint_name>lh_upper_leg_joint</joint_name>
+      <p_gain>200</p_gain>
+      <i_gain>0.01</i_gain>
+      <d_gain>10</d_gain>
+      <cmd_max>33.5</cmd_max>
+      <cmd_min>-33.5</cmd_min>
+    </plugin>
+  </gazebo>
+  <gazebo>
+    <plugin filename="gz-sim-joint-position-controller-system"
+            name="gz::sim::systems::JointPositionController">
+      <joint_name>lh_lower_leg_joint</joint_name>
+      <p_gain>200</p_gain>
+      <i_gain>0.01</i_gain>
+      <d_gain>10</d_gain>
+      <cmd_max>33.5</cmd_max>
+      <cmd_min>-33.5</cmd_min>
+    </plugin>
+  </gazebo>
+  <gazebo>
+    <plugin filename="gz-sim-joint-position-controller-system"
+            name="gz::sim::systems::JointPositionController">
+      <joint_name>rh_hip_joint</joint_name>
+      <p_gain>200</p_gain>
+      <i_gain>0.01</i_gain>
+      <d_gain>10</d_gain>
+      <cmd_max>33.5</cmd_max>
+      <cmd_min>-33.5</cmd_min>
+    </plugin>
+  </gazebo>
+  <gazebo>
+    <plugin filename="gz-sim-joint-position-controller-system"
+            name="gz::sim::systems::JointPositionController">
+      <joint_name>rh_upper_leg_joint</joint_name>
+      <p_gain>200</p_gain>
+      <i_gain>0.01</i_gain>
+      <d_gain>10</d_gain>
+      <cmd_max>33.5</cmd_max>
+      <cmd_min>-33.5</cmd_min>
+    </plugin>
+  </gazebo>
+  <gazebo>
+    <plugin filename="gz-sim-joint-position-controller-system"
+            name="gz::sim::systems::JointPositionController">
+      <joint_name>rh_lower_leg_joint</joint_name>
+      <p_gain>200</p_gain>
+      <i_gain>0.01</i_gain>
+      <d_gain>10</d_gain>
+      <cmd_max>33.5</cmd_max>
+      <cmd_min>-33.5</cmd_min>
+    </plugin>
+  </gazebo>
 </xacro:macro>
 </robot>
+<!-- This file is appended to by the setup script -->
